File: hardware/Solaria/Solaria.kicad_sch (KiCad schematic)
At the start: 26 parts, among them J1 BATERIAS, J2 PANELSOLAR, J3 CONTROLVCC, Q1 2N3904, Q2 IRF9540N, Q3 2N3904, Q4 IRF9540N, Q5 IRF9540N, Q6 2N3904, Q7 2N3904, Q8 IRF9540N, U1 TP4056, U2 TP4056, U3 LM2596, U4 MT3608

Commit message: feat: añadido de hardware, docs y firmware de ultima version
Parts:
- added SW1: SW_DPST_x2, Button_Switch_THT:SW_PUSH-12mm_Wuerth-430476085716, symbol Switch:SW_DPST_x2
Connections:
- net at D3.1 (K), D4.1 (K), U4.1 (VIN+): now also SW1.1 (A)
- net at Q5.3 (S), R5.2, U1.3 (OUT+): now also SW1.2 (B)
Changed lines of the file:
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@@
 	)
 	(junction
+		(at 111.76 130.81)
+		(diameter 0)
+		(color 0 0 0 0)
+	)
+	(junction
 		(at 148.59 130.81)
 		(diameter 0)
@@
 	)
 	(junction
+		(at 111.76 101.6)
+		(diameter 0)
+		(color 0 0 0 0)
+	)
+	(junction
 		(at 135.89 66.04)
 		(diameter 0)
@@
 	(wire
 		(pts
+			(xy 48.26 130.81) (xy 111.76 130.81)
+		)
+		(stroke
+			(width 0)
+			(type default)
+		)
+	)
+	(wire
+		(pts
 			(xy 179.07 66.04) (xy 175.26 66.04)
 		)
@@
 	(wire
 		(pts
+			(xy 48.26 118.11) (xy 48.26 130.81)
+		)
+		(stroke
+			(width 0)
+			(type default)
+		)
+	)
+	(wire
+		(pts
 			(xy 187.96 66.04) (xy 200.66 66.04)
 		)
@@
 	(wire
 		(pts
+			(xy 48.26 107.95) (xy 48.26 101.6)
+		)
+		(stroke
+			(width 0)
+			(type default)
+		)
+	)
+	(wire
+		(pts
 			(xy 166.37 63.5) (xy 175.26 63.5)
 		)
@@
 	(wire
 		(pts
+			(xy 48.26 101.6) (xy 111.76 101.6)
+		)
+		(stroke
+			(width 0)
+			(type default)
+		)
+	)
+	(wire
+		(pts
 			(xy 99.06 107.95) (xy 86.36 107.95)
 		)
@@
 					(unit 1)
 				)
+			)
+		)
+	)
+	(symbol
+		(lib_id "Switch:SW_DPST_x2")
+		(at 48.26 113.03 90)
+		(unit 1)
+		(body_style 1)
+		(exclude_from_sim no)
+		(in_bom yes)
+		(on_board yes)
+		(in_pos_files yes)
+		(dnp no)
+		(fields_autoplaced yes)
+		(property "Reference" "SW1"
+			(at 49.53 111.7599 90)
+			(show_name no)
+			(do_not_autoplace no)
+			(effects
+				(font
+					(size 1.27 1.27)
+				)
+				(justify right)
+			)
+		)
+		(property "Value" "SW_DPST_x2"
+			(at 49.53 114.2999 90)
+			(show_name no)
+			(do_not_autoplace no)
+			(effects
+				(font
+					(size 1.27 1.27)
+				)
+				(justify right)
+			)
+		)
+		(property "Footprint" "Button_Switch_THT:SW_PUSH-12mm_Wuerth-430476085716"
+			(at 48.26 113.03 0)
+			(hide yes)
+			(show_name no)
+			(do_not_autoplace no)
+			(effects
+				(font
+					(size 1.27 1.27)
+				)
+			)
+		)
+		(property "Datasheet" ""
+			(at 48.26 113.03 0)
+			(hide yes)
+			(show_name no)
+			(do_not_autoplace no)
+			(effects
+				(font
+					(size 1.27 1.27)
+				)
+			)
+		)
+		(property "Description" "Single Pole Single Throw (SPST) switch, separate symbol"
+			(at 48.26 113.03 0)
+			(hide yes)
+			(show_name no)
+			(do_not_autoplace no)
+			(effects
+				(font
+					(size 1.27 1.27)
+				)
+			)
+		)
+		(pin "3"
+		)
+		(pin "2"
+		)
+		(pin "1"
+		)
+		(pin "4"
+		)
+		(instances
+			(project "sistemasolar"
+				(path "/37605b2f-a95c-4385-8c81-ccd587e35e25"
+					(reference "SW1")
+					(unit 1)
+				)
